Commit message: fix wrong urdf load, detects collision/contact events now

File: libraries/irobot_create_description/urdf/create_base.xacro (robot description, xacro)
@@ -20,27 +20,29 @@
     <xacro:property name="wheel_length" value="0.02" />
     <xacro:property name="caster_wheel_offset_y" value="0.17" />
-	<xacro:macro name="wheel_xmission" params="wheel_prefix">
-		<transmission name="${wheel_prefix}_wheel_trans">
-			<type>transmission_interface/SimpleTransmission</type>
-			<actuator name="${wheel_prefix}_wheel_motor">
-				<hardwareInterface>VelocityJointInterface</hardwareInterface>
-				<mechanicalReduction>1</mechanicalReduction>
-			</actuator>
-			<joint name="${wheel_prefix}_wheel_joint">
-				<hardwareInterface>VelocityJointInterface</hardwareInterface>
-			</joint>
-		</transmission>
-	</xacro:macro>
+    <xacro:macro name="wheel_xmission" params="wheel_prefix">
+        <transmission name="${wheel_prefix}_wheel_trans">
+            <type>transmission_interface/SimpleTransmission</type>
+            <actuator name="${wheel_prefix}_wheel_motor">
+                <hardwareInterface>VelocityJointInterface</hardwareInterface>
+                <mechanicalReduction>1</mechanicalReduction>
+            </actuator>
+            <joint name="${wheel_prefix}_wheel_joint">
+                <hardwareInterface>VelocityJointInterface</hardwareInterface>
+            </joint>
+        </transmission>
+    </xacro:macro>
     <xacro:macro name="create">
         <!-- base_footprint is a fictitious link(frame) that is on the ground right below base_link origin,
              navigation stack depends on this frame -->
         <link name="base_footprint">
+            <!--
             <inertial>
                 <mass value="0.0001" />
                 <origin xyz="0 0 0" />
                 <inertia ixx="0.0001" ixy="0.0" ixz="0.0"
-                         iyy="0.0001" iyz="0.0"
-                         izz="0.0001" />
-            </inertial>
+                    iyy="0.0001" iyz="0.0"
+                    izz="0.0001" />
+            </inertial>
+            -->
             <visual>
                 <origin xyz="0 0 0" rpy="0 0 0" />
@@ -53,5 +55,5 @@
                 <origin xyz="0 0 ${base_size_z/2 + 0.051}" rpy="0 0 0" />
                 <geometry>
-                  <box size="0.001 0.001 0.001" />
+                    <box size="0.001 0.001 0.001" />
                 </geometry>
             </collision>
@@ -70,6 +72,6 @@
                 <origin xyz="${-base_size_x/2} 0 ${-base_size_z/2}" />
                 <inertia ixx="1.0" ixy="0.0" ixz="0.0"
-                         iyy="1.0" iyz="0.0"
-                         izz="1.0" />
+                    iyy="1.0" iyz="0.0"
+                    izz="1.0" />
             </inertial>
             <visual>
@@ -101,6 +103,6 @@
                 <origin xyz="0 0 0" />
                 <inertia  ixx="0.012411765597" ixy="-0.000711733678" ixz="0.00050272983"
-                          iyy="0.015218160428" iyz="-0.000004273467"
-                          izz="0.011763977943" />
+                    iyy="0.015218160428" iyz="-0.000004273467"
+                    izz="0.011763977943" />
             </inertial>
             <visual>
@@ -146,6 +148,6 @@
                 <origin xyz="0 0 0" />
                 <inertia ixx="0.01" ixy="0.0" ixz="0.0"
-                         iyy="0.01" iyz="0.0"
-                         izz="0.01" />
+                    iyy="0.01" iyz="0.0"
+                    izz="0.01" />
             </inertial>
             <visual>
@@ -184,6 +186,6 @@
                 <origin xyz="0 0 0" rpy="0 0 0" />
                 <inertia  ixx="0.012411765597" ixy="-0.000711733678" ixz="0.00050272983"
-                          iyy="0.015218160428" iyz="-0.000004273467"
-                          izz="0.011763977943" />
+                    iyy="0.015218160428" iyz="-0.000004273467"
+                    izz="0.011763977943" />
             </inertial>
             <visual>
@@ -194,8 +196,8 @@
             </visual>
             <collision>
-            <origin xyz="0 0 0" rpy="${M_PI/2} 0 0" />
-            <geometry>
+                <origin xyz="0 0 0" rpy="${M_PI/2} 0 0" />
+                <geometry>
                     <cylinder radius="0.007" length="0.015" />
-            </geometry>
+                </geometry>
             </collision>
         </link>
@@ -239,4 +241,20 @@
             </plugin>
         </gazebo>
+        <!-- Contact -->
+        <gazebo reference="base_link">
+            <sensor name="bumper" type="contact">
+                <always_on>true</always_on>
+                <update_rate>50</update_rate>
+                <contact>
+                    <collision>base_footprint_fixed_joint_lump__base_link_collision_1</collision>
+                </contact>
+                <plugin name="base_link_bumper" filename="libgazebo_ros_bumper.so">
+                    <alwaysOn>true</alwaysOn>
+                    <updateRate>50</updateRate>
+                    <bumperTopicName>$(arg ns)/bumper</bumperTopicName>
+                    <frameName>$(arg ns)</frameName>
+                </plugin>
+            </sensor>
+        </gazebo>
         <!-- GAZEBO MATERIALS -->
         <gazebo reference="base_link">

Commit message: new urdf, because the old one was very inaccurate and unwieldy. Works.

File: libraries/irobot_create_description/urdf/create_base.xacro (robot description, xacro)
@@ -19,5 +19,5 @@
     <xacro:property name="wheel_radius" value="0.0346" />
     <xacro:property name="wheel_length" value="0.02" />
-    <xacro:property name="caster_wheel_offset_y" value="0.17" />
+    <xacro:property name="wheel_separation" value="0.26" />
     <xacro:macro name="wheel_xmission" params="wheel_prefix">
         <transmission name="${wheel_prefix}_wheel_trans">
@@ -28,5 +28,5 @@
             </actuator>
             <joint name="${wheel_prefix}_wheel_joint">
-                <hardwareInterface>VelocityJointInterface</hardwareInterface>
+                <hardwareInterface>hardware_interface/VelocityJointInterface</hardwareInterface>
             </joint>
         </transmission>
@@ -53,5 +53,5 @@
             </visual>
             <collision>
-                <origin xyz="0 0 ${base_size_z/2 + 0.051}" rpy="0 0 0" />
+                <origin xyz="0 0 0" rpy="0 0 0" />
                 <geometry>
                     <box size="0.001 0.001 0.001" />
@@ -62,5 +62,5 @@
             <!-- NB: While you would think this would make it go up, it is oddly reversed.
                  This moves the joint to 0,0,0 where we want it for rviz, etc. -->
-            <origin xyz="0 0 ${base_size_z/2 + 0.051}" rpy="0 0 0" />
+            <origin xyz="0 0 ${base_size_z/2-0.051}" rpy="0 0 0" />
             <parent link="base_footprint"/>
             <child link="base_link" />
@@ -69,6 +69,6 @@
         <link name="base_link">
             <inertial>
-                <mass value="12" />
-                <origin xyz="${-base_size_x/2} 0 ${-base_size_z/2}" />
+                <mass value="3.58" />
+                <origin xyz="${-base_size_x/2} 0 ${base_size_z/2}" />
                 <inertia ixx="1.0" ixy="0.0" ixz="0.0"
                     iyy="1.0" iyz="0.0"
@@ -145,5 +145,5 @@
         <link name="base_caster_support_link">
             <inertial>
-                <mass value="25.0"/>
+                <mass value="5.0"/>
                 <origin xyz="0 0 0" />
                 <inertia ixx="0.01" ixy="0.0" ixz="0.0"
@@ -228,5 +228,5 @@
                 <legacyMode>false</legacyMode>
                 <!-- Config -->
-                <wheelSeparation>${caster_wheel_offset_y*2}</wheelSeparation>
+                <wheelSeparation>${wheel_separation}</wheelSeparation>
                 <wheelDiameter>${wheel_radius*2}</wheelDiameter>
                 <wheelAcceleration>0</wheelAcceleration>
@@ -240,4 +240,11 @@
                 <!-- Odometry Source?? -->
             </plugin>
+            <!--
+            <plugin name="gazebo_ros_control" filename="libgazebo_ros_control.so">
+                <robotNamespace>$(arg ns)</robotNamespace>
+                <robotSimType>gazebo_ros_control/DefaultRobotHWSim</robotSimType>
+                <robotParam>$(arg ns)/urdf</robotParam>
+            </plugin>
+            -->
         </gazebo>
         <!-- Contact -->
