Commit message: added top plate and verified collision still works

File: libraries/irobot_create_description/urdf/common.xacro (robot description, xacro)
@@ -2,5 +2,5 @@
 <robot
   xmlns:xacro="http://ros.org/wiki/xacro">
-  <property name="M_PI" value="3.1415926535897931" />
+  <xacro:property name="M_PI" value="3.1415926535897931" />
   <!-- see https://secure.wikimedia.org/wikipedia/en/wiki/List_of_moment_of_inertia_tensors -->
   <!-- #################### versions without origin #################### -->
@@ -36,5 +36,5 @@
     <inertial>
       <mass value="${mass}" />
-      <insert_block name="origin" />
+      <xacro:insert_block name="origin" />
       <inertia ixx="${0.4 * mass * radius * radius}" ixy="0.0" ixz="0.0"
         iyy="${0.4 * mass * radius * radius}" iyz="0.0"
@@ -45,5 +45,5 @@
     <inertial>
       <mass value="${mass}" />
-      <insert_block name="origin" />
+      <xacro:insert_block name="origin" />
       <inertia ixx="${0.0833333 * mass * (3 * radius * radius + length * length)}" ixy="0.0" ixz="0.0"
         iyy="${0.0833333 * mass * (3 * radius * radius + length * length)}" iyz="0.0"
@@ -54,5 +54,5 @@
     <inertial>
       <mass value="${mass}" />
-      <insert_block name="origin" />
+      <xacro:insert_block name="origin" />
       <inertia ixx="${0.0833333 * mass * (y*y + z*z)}" ixy="0.0" ixz="0.0"
         iyy="${0.0833333 * mass * (x*x + z*z)}" iyz="0.0"

File: libraries/irobot_create_description/urdf/roomba.urdf.xacro (robot description, xacro)
@@ -1,4 +1,5 @@
 <?xml version="1.0"?>
 <robot name="roomba" xmlns:xacro="http://ros.org/wiki/xacro">
+    <xacro:include filename="$(find irobot_create_description)/urdf/top_plate.urdf.xacro" />
     <xacro:arg name="ns" default="target0"/>
     <xacro:arg name="color" default="white"/>
@@ -10,4 +11,5 @@
     <xacro:property name="ns" value="$(arg ns)"/>
     <xacro:property name="obs" value="${ns.startswith('obs')}" />
+    <xacro:property name="pole" value="$(arg pole)"/>
     <xacro:macro name="wheel_xmission" params="wheel_prefix">
         <transmission name="${wheel_prefix}_wheel_trans">
@@ -221,4 +223,7 @@
     </joint>
     <xacro:unless value="${obs}">
+        <!-- random color -->
+        <top_plate parent="base_link" height="0.125" red="${(pole % 0.034) >= 0.017}"/>
+        <!--
         <link name="top_tap_link">
             <collision>
@@ -234,4 +239,5 @@
             <child link="top_tap_link"/>
         </joint>
+        -->
     </xacro:unless>
     <!-- wheels and caster wheel -->
@@ -324,13 +330,13 @@
             </inertial>
             <visual>
-                <origin xyz="0 0 ${$(arg pole)/2.0}" rpy="0 0 0"/>
+                <origin xyz="0 0 ${pole/2.0}" rpy="0 0 0"/>
                 <geometry>
-                    <cylinder length="$(arg pole)" radius="0.05"/>
+                    <cylinder length="${pole}" radius="0.05"/>
                 </geometry>
             </visual>
             <collision>
-                <origin xyz="0 0 ${$(arg pole)/2.0}" rpy="0 0 0"/>
+                <origin xyz="0 0 ${pole/2.0}" rpy="0 0 0"/>
                 <geometry>
-                    <cylinder length="$(arg pole)" radius="0.05"/>
+                    <cylinder length="${pole}" radius="0.05"/>
                 </geometry>
             </collision>
@@ -385,5 +391,5 @@
             <plugin name="target_roomba" filename="libtarget_roomba.so">
                 <front_bumper>front_bumper_link</front_bumper>
-                <top_tap>top_tap_link</top_tap>
+                <top_tap>top_plate_link</top_tap>
                 <wheel_separation>${wheel_separation}</wheel_separation>
                 <wheel_radius>${wheel_radius}</wheel_radius>
@@ -413,5 +419,5 @@
     </gazebo>
     <xacro:unless value="${obs}">
-        <gazebo reference="top_tap_link">
+        <gazebo reference="top_plate_link">
             <sensor name="top_tap" type="contact">
                 <always_on>true</always_on>
@@ -419,5 +425,5 @@
                 <contact>
                     <!-- unfortunately, gazebo lumps fixed joints into ridiculous names -->
-                    <collision>base_footprint_fixed_joint_lump__top_tap_link_collision_4</collision>
+                    <collision>base_footprint_fixed_joint_lump__top_plate_link_collision_4</collision>
                 </contact>
                 <plugin name="top_tap" filename="libgazebo_ros_bumper.so">
