Commit message: obstacle roomba stuff

File: libraries/irobot_create_description/urdf/roomba.urdf.xacro (robot description, xacro)
@@ -3,4 +3,5 @@
     <xacro:arg name="ns" default="target0"/>
     <xacro:arg name="color" default="white"/>
+    <xacro:arg name="obs" default="false"/>
     <xacro:property name="M_PI" value="3.14159"/>
     <xacro:property name="wheel_radius" value="0.033" />
@@ -311,4 +312,26 @@
     <wheel_xmission wheel_prefix="left"/>
     <wheel_xmission wheel_prefix="right"/>
+    <xacro:if value="$(arg obs)">
+        <link name="pole_link">
+            <visual>
+                <origin xyz="0 0 0" rpy="0 0 0"/>
+                <geometry>
+                    <cylinder length="1.0" radius="0.05"/>
+                </geometry>
+            </visual>
+            <collision>
+                <origin xyz="0 0 0" rpy="0 0 0"/>
+                <geometry>
+                    <cylinder length="1.0" radius="0.05"/>
+                </geometry>
+            </collision>
+        </link>
+        <joint name="pole_joint" type="fixed">
+            <origin xyz="0 0 0.0" rpy="0 0 0"/>
+            <parent link="base_link"/>
+            <child link="pole_link"/>
+            <axis xyz="0 0 1"/>
+        </joint>
+    </xacro:if>
     <gazebo>
         <!--
@@ -336,14 +359,29 @@
         </plugin>
         -->
-        <plugin name="target_roomba" filename="libtarget_roomba.so">
-            <front_bumper>base_footprint_fixed_joint_lump__front_bumper_link_collision_3</front_bumper>
-            <top_tap>base_footprint_fixed_joint_lump__top_tap_link_collision_4</top_tap>
-            <wheel_separation>${wheel_separation}</wheel_separation>
-            <wheel_radius>${wheel_radius}</wheel_radius>
-            <left_joint>left_wheel_joint</left_joint>
-            <right_joint>right_wheel_joint</right_joint>
-            <lin_vel>0.33</lin_vel>
-            <ang_vel>1.375</ang_vel>
-        </plugin>
+        <xacro:if value="$(arg obs)">
+            <plugin name="obstacle_roomba" filename="libobstacle_roomba.so">
+                <front_bumper>base_footprint_fixed_joint_lump__front_bumper_link_collision_3</front_bumper>
+                <pole_link>pole_link</pole_link>
+                <!--<top_tap>base_footprint_fixed_joint_lump__top_tap_link_collision_4</top_tap>-->
+                <wheel_separation>${wheel_separation}</wheel_separation>
+                <wheel_radius>${wheel_radius}</wheel_radius>
+                <left_joint>left_wheel_joint</left_joint>
+                <right_joint>right_wheel_joint</right_joint>
+                <lin_vel>0.33</lin_vel>
+                <ang_vel>0.066</ang_vel>
+            </plugin>
+        </xacro:if>
+        <xacro:unless value="$(arg obs)">
+            <plugin name="target_roomba" filename="libtarget_roomba.so">
+                <front_bumper>base_footprint_fixed_joint_lump__front_bumper_link_collision_3</front_bumper>
+                <top_tap>base_footprint_fixed_joint_lump__top_tap_link_collision_4</top_tap>
+                <wheel_separation>${wheel_separation}</wheel_separation>
+                <wheel_radius>${wheel_radius}</wheel_radius>
+                <left_joint>left_wheel_joint</left_joint>
+                <right_joint>right_wheel_joint</right_joint>
+                <lin_vel>0.33</lin_vel>
+                <ang_vel>1.375</ang_vel>
+            </plugin>
+        </xacro:unless>
     </gazebo>
     <gazebo reference="front_bumper_link">
@@ -363,19 +401,21 @@
         </sensor>
     </gazebo>
-    <gazebo reference="top_tap_link">
-        <sensor name="top_tap" type="contact">
-            <always_on>true</always_on>
-            <update_rate>50</update_rate>
-            <contact>
-                <!-- unfortunately, urdf->xacro lumps fixed joints into ridiculous names -->.
-                <collision>base_footprint_fixed_joint_lump__top_tap_link_collision_4</collision>
-            </contact>
-            <plugin name="top_tap" filename="libgazebo_ros_bumper.so">
-                <alwaysOn>true</alwaysOn>
-                <updateRate>50</updateRate>
-                <bumperTopicName>$(arg ns)/top_tap</bumperTopicName>
-                <frameName>$(arg ns)</frameName>
-            </plugin>
-        </sensor>
-    </gazebo>
+    <xacro:if value="$(arg obs)">
+        <gazebo reference="top_tap_link">
+            <sensor name="top_tap" type="contact">
+                <always_on>true</always_on>
+                <update_rate>50</update_rate>
+                <contact>
+                    <!-- unfortunately, urdf->xacro lumps fixed joints into ridiculous names -->.
+                    <collision>base_footprint_fixed_joint_lump__top_tap_link_collision_4</collision>
+                </contact>
+                <plugin name="top_tap" filename="libgazebo_ros_bumper.so">
+                    <alwaysOn>true</alwaysOn>
+                    <updateRate>50</updateRate>
+                    <bumperTopicName>$(arg ns)/top_tap</bumperTopicName>
+                    <frameName>$(arg ns)</frameName>
+                </plugin>
+            </sensor>
+        </gazebo>
+    </xacro:if>
 </robot>

Commit message: bug with no collision detection?

File: libraries/irobot_create_description/urdf/roomba.urdf.xacro (robot description, xacro)
@@ -218,17 +218,19 @@
         <child link="front_bumper_link"/>
     </joint>
-    <link name="top_tap_link">
-        <collision>
-            <origin xyz="0.0 0.0 0.1" rpy="0 0 0" />
-            <geometry>
-                <cylinder length="0.01" radius="0.15"/>
-            </geometry>
-        </collision>
-    </link>
-    <joint name="top_tap_joint" type="fixed">
-        <origin xyz="0 0 0" rpy="0 0 0"/>
-        <parent link="base_link"/>
-        <child link="top_tap_link"/>
-    </joint>
+    <xacro:unless value="$(arg obs)">
+        <link name="top_tap_link">
+            <collision>
+                <origin xyz="0.0 0.0 0.1" rpy="0 0 0" />
+                <geometry>
+                    <cylinder length="0.01" radius="0.15"/>
+                </geometry>
+            </collision>
+        </link>
+        <joint name="top_tap_joint" type="fixed">
+            <origin xyz="0 0 0" rpy="0 0 0"/>
+            <parent link="base_link"/>
+            <child link="top_tap_link"/>
+        </joint>
+    </xacro:unless>
     <!-- wheels and caster wheel -->
     <link name="left_wheel_link">
@@ -315,5 +317,5 @@
         <link name="pole_link">
             <visual>
-                <origin xyz="0 0 0" rpy="0 0 0"/>
+                <origin xyz="0 0 0.5" rpy="0 0 0"/>
                 <geometry>
                     <cylinder length="1.0" radius="0.05"/>
@@ -321,5 +323,5 @@
             </visual>
             <collision>
-                <origin xyz="0 0 0" rpy="0 0 0"/>
+                <origin xyz="0 0 0.5" rpy="0 0 0"/>
                 <geometry>
                     <cylinder length="1.0" radius="0.05"/>
@@ -328,5 +330,5 @@
         </link>
         <joint name="pole_joint" type="fixed">
-            <origin xyz="0 0 0.0" rpy="0 0 0"/>
+            <origin xyz="0 0 0.082" rpy="0 0 0"/>
             <parent link="base_link"/>
             <child link="pole_link"/>
@@ -390,5 +392,5 @@
             <update_rate>50</update_rate>
             <contact>
-                <!-- unfortunately, urdf->xacro lumps fixed joints into ridiculous names -->.
+                <!-- unfortunately, gazebo lumps fixed joints into ridiculous names -->.
                 <collision>base_footprint_fixed_joint_lump__front_bumper_link_collision_3</collision>
             </contact>
@@ -401,5 +403,5 @@
         </sensor>
     </gazebo>
-    <xacro:if value="$(arg obs)">
+    <xacro:unless value="$(arg obs)">
         <gazebo reference="top_tap_link">
             <sensor name="top_tap" type="contact">
@@ -407,5 +409,5 @@
                 <update_rate>50</update_rate>
                 <contact>
-                    <!-- unfortunately, urdf->xacro lumps fixed joints into ridiculous names -->.
+                    <!-- unfortunately, gazebo lumps fixed joints into ridiculous names -->.
                     <collision>base_footprint_fixed_joint_lump__top_tap_link_collision_4</collision>
                 </contact>
@@ -418,4 +420,4 @@
             </sensor>
         </gazebo>
-    </xacro:if>
+    </xacro:unless>
 </robot>

Commit message: it is simply impossible to set random pole height. generating instead.

File: libraries/irobot_create_description/urdf/roomba.urdf.xacro (robot description, xacro)
@@ -3,9 +3,11 @@
     <xacro:arg name="ns" default="target0"/>
     <xacro:arg name="color" default="white"/>
-    <xacro:arg name="obs" default="false"/>
+    <xacro:arg name="pole" default="1.0"/>
     <xacro:property name="M_PI" value="3.14159"/>
     <xacro:property name="wheel_radius" value="0.033" />
     <xacro:property name="wheel_length" value="0.023" />
     <xacro:property name="wheel_separation" value="0.24" />
+    <xacro:property name="ns" value="$(arg ns)"/>
+    <xacro:property name="obs" value="${ns.startswith('obs')}" />
     <xacro:macro name="wheel_xmission" params="wheel_prefix">
         <transmission name="${wheel_prefix}_wheel_trans">
@@ -218,5 +220,5 @@
         <child link="front_bumper_link"/>
     </joint>
-    <xacro:unless value="$(arg obs)">
+    <xacro:unless value="${obs}">
         <link name="top_tap_link">
             <collision>
@@ -314,21 +316,27 @@
     <wheel_xmission wheel_prefix="left"/>
     <wheel_xmission wheel_prefix="right"/>
-    <xacro:if value="$(arg obs)">
+    <xacro:if value="${obs}">
         <link name="pole_link">
+            <gravity>true</gravity>
+            <inertial>
+                <mass value="0.01" />
+                <origin xyz="0 0 0" />
+                <inertia ixx="0.01" ixy="0.0" ixz="0.0" iyy="0.01" iyz="0.0" izz="0.5" />
+            </inertial>
             <visual>
-                <origin xyz="0 0 0.5" rpy="0 0 0"/>
+                <origin xyz="0 0 ${$(arg pole)/2.0}" rpy="0 0 0"/>
                 <geometry>
-                    <cylinder length="1.0" radius="0.05"/>
+                    <cylinder length="$(arg pole)" radius="0.05"/>
                 </geometry>
             </visual>
             <collision>
-                <origin xyz="0 0 0.5" rpy="0 0 0"/>
+                <origin xyz="0 0 ${$(arg pole)/2.0}" rpy="0 0 0"/>
                 <geometry>
-                    <cylinder length="1.0" radius="0.05"/>
+                    <cylinder length="$(arg pole)" radius="0.05"/>
                 </geometry>
             </collision>
         </link>
         <joint name="pole_joint" type="fixed">
-            <origin xyz="0 0 0.082" rpy="0 0 0"/>
+            <origin xyz="0 0 0.0358" rpy="0 0 0"/>
             <parent link="base_link"/>
             <child link="pole_link"/>
@@ -361,5 +369,5 @@
         </plugin>
         -->
-        <xacro:if value="$(arg obs)">
+        <xacro:if value="${obs}">
             <plugin name="obstacle_roomba" filename="libobstacle_roomba.so">
                 <front_bumper>base_footprint_fixed_joint_lump__front_bumper_link_collision_3</front_bumper>
@@ -374,5 +382,5 @@
             </plugin>
         </xacro:if>
-        <xacro:unless value="$(arg obs)">
+        <xacro:unless value="${obs}">
             <plugin name="target_roomba" filename="libtarget_roomba.so">
                 <front_bumper>front_bumper_link</front_bumper>
@@ -403,5 +411,5 @@
         </sensor>
     </gazebo>
-    <xacro:unless value="$(arg obs)">
+    <xacro:unless value="${obs}">
         <gazebo reference="top_tap_link">
             <sensor name="top_tap" type="contact">

Commit message: remove deprecated crap

File: libraries/irobot_create_description/urdf/roomba.urdf.xacro (robot description, xacro)
@@ -61,150 +61,4 @@
         <child link="base_link" />
     </joint>
-    <!-- Ignore Unused Sensors
-    <link name="left_cliff_sensor_link">
-        <inertial>
-            <mass value="0.01" />
-            <origin xyz="0 0 0"/>
-            <inertia ixx="0.001" ixy="0.0" ixz="0.0" iyy="0.001" iyz="0.0" izz="0.001" />
-        </inertial>
-    </link>
-    <link name="right_cliff_sensor_link">
-        <inertial>
-            <mass value="0.01" />
-            <origin xyz="0 0 0"/>
-            <inertia ixx="0.001" ixy="0.0" ixz="0.0" iyy="0.001" iyz="0.0" izz="0.001" />
-        </inertial>
-    </link>
-    <link name="front_left_cliff_sensor_link">
-        <inertial>
-            <mass value="0.01" />
-            <origin xyz="0 0 0"/>
-            <inertia ixx="1.0" ixy="0.0" ixz="0.0" iyy="0.01" iyz="0.0" izz="0.01" />
-        </inertial>
-    </link>
-    <link name="front_right_cliff_sensor_link">
-        <inertial>
-            <mass value="0.01" />
-            <origin xyz="0 0 0"/>
-            <inertia ixx="0.001" ixy="0.0" ixz="0.0" iyy="0.001" iyz="0.0" izz="0.001" />
-        </inertial>
-    </link>
-    <joint name="left_sensor_joint" type="fixed">
-        <origin xyz="0.07 0.14 0.01" rpy="0 1.57079 0" />
-        <parent link="base_link"/>
-        <child link="left_cliff_sensor_link" />
-    </joint>
-    <joint name="right_cliff_sensor_joint" type="fixed">
-        <origin xyz="0.07 -0.14 0.01" rpy="0 1.57079 0" />
-        <parent link="base_link"/>
-        <child link="right_cliff_sensor_link" />
-    </joint>
-    <joint name="front_left_cliff_sensor_joint" type="fixed">
-        <origin xyz="0.15 0.04 0.01" rpy="0 1.57079 0" />
-        <parent link="base_link"/>
-        <child link="front_left_cliff_sensor_link" />
-    </joint>
-    <joint name="front_right_cliff_sensor_joint" type="fixed">
-        <origin xyz="0.15 -0.04 0.01" rpy="0 1.57079 0" />
-        <parent link="base_link"/>
-        <child link="front_right_cliff_sensor_link" />
-    </joint>
-    <link name="left_ir_sensor_link">
-        <inertial>
-            <mass value="0.01" />
-            <origin xyz="0 0 0"/>
-            <inertia ixx="0.001" ixy="0.0" ixz="0.0" iyy="0.001" iyz="0.0" izz="0.001" />
-        </inertial>
-    </link>
-    <link name="front_left_ir_sensor_link">
-        <inertial>
-            <mass value="0.01" />
-            <origin xyz="0 0 0"/>
-            <inertia ixx="0.001" ixy="0.0" ixz="0.0" iyy="0.001" iyz="0.0" izz="0.001" />
-        </inertial>
-    </link>
-    <link name="center_left_ir_sensor_link">
-        <inertial>
-            <mass value="0.01" />
-            <origin xyz="0 0 0"/>
-            <inertia ixx="0.001" ixy="0.0" ixz="0.0" iyy="0.001" iyz="0.0" izz="0.001" />
-        </inertial>
-    </link>
-    <link name="center_right_ir_sensor_link">
-        <inertial>
-            <mass value="0.01" />
-            <origin xyz="0 0 0"/>
-            <inertia ixx="0.001" ixy="0.0" ixz="0.0" iyy="0.001" iyz="0.0" izz="0.001" />
-        </inertial>
-    </link>
-    <link name="front_right_ir_sensor_link">
-        <inertial>
-            <mass value="0.01" />
-            <origin xyz="0 0 0"/>
-            <inertia ixx="0.001" ixy="0.0" ixz="0.0" iyy="0.001" iyz="0.0" izz="0.001" />
-        </inertial>
-    </link>
-    <link name="right_ir_sensor_link">
-        <inertial>
-            <mass value="0.01" />
-            <origin xyz="0 0 0"/>
-            <inertia ixx="0.001" ixy="0.0" ixz="0.0" iyy="0.001" iyz="0.0" izz="0.001" />
-        </inertial>
-    </link>
-    <joint name="left_ir_sensor_joint" type="fixed">
-        <origin xyz="0.01 0.15 0.042" rpy="0 0 1.5" />
-        <parent link="base_link"/>
-        <child link="left_ir_sensor_link" />
-    </joint>
-    <joint name="front_left_ir_sensor_joint" type="fixed">
-        <origin xyz="0.09 0.12 0.042" rpy="0 0 1.0" />
-        <parent link="base_link"/>
-        <child link="front_left_ir_sensor_link" />
-    </joint>
-    <joint name="center_left_ir_sensor_joint" type="fixed">
-        <origin xyz="0.15 0.04 0.042" rpy="0 0 0.4" />
-        <parent link="base_link"/>
-        <child link="center_left_ir_sensor_link" />
-    </joint>
-    <joint name="center_right_ir_sensor_joint" type="fixed">
-        <origin xyz="0.15 -0.04 0.042" rpy="0 0 -0.4" />
-        <parent link="base_link"/>
-        <child link="center_right_ir_sensor_link" />
-    </joint>
-    <joint name="front_right_ir_sensor_joint" type="fixed">
-        <origin xyz="0.09 -0.120 0.042" rpy="0 0 -1.0" />
-        <parent link="base_link"/>
-        <child link="front_right_ir_sensor_link" />
-    </joint>
-    <joint name="right_ir_sensor_joint" type="fixed">
-        <origin xyz="0.01 -0.15 0.042" rpy="0 0 -1.5" />
-        <parent link="base_link"/>
-        <child link="right_ir_sensor_link" />
-    </joint>
-    <link name="left_bumper_link">
-        <inertial>
-            <mass value="0.01" />
-            <origin xyz="0 0 0"/>
-            <inertia ixx="0.001" ixy="0.0" ixz="0.0" iyy="0.001" iyz="0.0" izz="0.001" />
-        </inertial>
-    </link>
-    <link name="right_bumper_link">
-        <inertial>
-            <mass value="0.01" />
-            <origin xyz="0 0 0"/>
-            <inertia ixx="0.001" ixy="0.0" ixz="0.0" iyy="0.001" iyz="0.0" izz="0.001" />
-        </inertial>
-    </link>
-    <joint name="left_bumper_joint" type="fixed">
-        <origin xyz="0.115 -0.115 0.042" rpy="0 0 -0.75" />
-        <parent link="base_link"/>
-        <child link="left_bumper_link" />
-    </joint>
-    <joint name="right_bumper_joint" type="fixed">
-        <origin xyz="0.115 0.115 0.042" rpy="0 0 0.75" />
-        <parent link="base_link"/>
-        <child link="right_bumper_link" />
-    </joint>
-    -->
     <!-- Collision Detections -->
     <link name="front_bumper_link">
@@ -225,19 +79,4 @@
         <!-- random color -->
         <top_plate parent="base_link" height="0.125" red="${(pole % 0.034) >= 0.017}"/>
-        <!--
-        <link name="top_tap_link">
-            <collision>
-                <origin xyz="0.0 0.0 0.1" rpy="0 0 0" />
-                <geometry>
-                    <cylinder length="0.01" radius="0.15"/>
-                </geometry>
-            </collision>
-        </link>
-        <joint name="top_tap_joint" type="fixed">
-            <origin xyz="0 0 0" rpy="0 0 0"/>
-            <parent link="base_link"/>
-            <child link="top_tap_link"/>
-        </joint>
-        -->
     </xacro:unless>
     <!-- wheels and caster wheel -->
@@ -350,28 +189,4 @@
     </xacro:if>
     <gazebo>
-        <!--
-       <plugin name="differential_drive_controller" filename="libgazebo_ros_diff_drive.so">
-            <alwaysOn>true</alwaysOn>
-            <update>100</update>
-            <robotNamespace>$(arg ns)</robotNamespace>
-            <commandTopic>cmd_vel</commandTopic>
-            <odometryTopic>odom</odometryTopic>
-            <odometryFrame>odom</odometryFrame>
-            <robotBaseFrame>base_link</robotBaseFrame>
-            <publishWheelTF>false</publishWheelTF>
-            <publishWheelJointState>false</publishWheelJointState>
-            <legacyMode>false</legacyMode>
-            <wheelSeparation>${wheel_separation}</wheelSeparation>
-            <wheelDiameter>${wheel_radius*2}</wheelDiameter>
-            <wheelAcceleration>0</wheelAcceleration>
-            <wheelTorque>50</wheelTorque>
-            <updateRate>100.0</updateRate>
-            <leftJoint>left_wheel_joint</leftJoint>
-            <rightJoint>right_wheel_joint</rightJoint>
-            <rosDebugLevel>na</rosDebugLevel>
-            <publishTf>true</publishTf>
-            <tf_prefix>$(arg ns)</tf_prefix>
-        </plugin>
-        -->
         <xacro:if value="${obs}">
             <plugin name="obstacle_roomba" filename="libobstacle_roomba.so">

Commit message: turns out, no reason to supply the god-awful collision link names in urdf (model plugin handles it)

File: libraries/irobot_create_description/urdf/roomba.urdf.xacro (robot description, xacro)
@@ -217,37 +217,3 @@
         </xacro:unless>
     </gazebo>
-    <gazebo reference="front_bumper_link">
-        <sensor name="front_bumper" type="contact">
-            <always_on>true</always_on>
-            <update_rate>50</update_rate>
-            <contact>
-                <!-- unfortunately, gazebo lumps fixed joints into ridiculous names -->
-                <collision>base_footprint_fixed_joint_lump__front_bumper_link_collision_3</collision>
-            </contact>
-            <plugin name="front_bumper" filename="libgazebo_ros_bumper.so">
-                <alwaysOn>true</alwaysOn>
-                <updateRate>50</updateRate>
-                <bumperTopicName>${ns}/front_bumper</bumperTopicName>
-                <frameName>${ns}</frameName>
-            </plugin>
-        </sensor>
-    </gazebo>
-    <xacro:unless value="${obs}">
-        <gazebo reference="top_plate_link">
-            <sensor name="top_tap" type="contact">
-                <always_on>true</always_on>
-                <update_rate>50</update_rate>
-                <contact>
-                    <!-- unfortunately, gazebo lumps fixed joints into ridiculous names -->
-                    <collision>base_footprint_fixed_joint_lump__top_plate_link_collision_4</collision>
-                </contact>
-                <plugin name="top_tap" filename="libgazebo_ros_bumper.so">
-                    <alwaysOn>true</alwaysOn>
-                    <updateRate>50</updateRate>
-                    <bumperTopicName>${ns}/top_tap</bumperTopicName>
-                    <frameName>${ns}</frameName>
-                </plugin>
-            </sensor>
-        </gazebo>
-    </xacro:unless>
 </robot>
