File: hardware/roomba_pcb/roomba_pcb.sch (KiCad schematic (older format))
At the start: 21 parts, among them J1 RECEIVER, J2 TO_CREATE, P1 Power, P2 Analog, P3 Digital, P4 Digital, P5 CONN_01X01, P6 CONN_01X01, P7 CONN_01X01, P8 CONN_01X01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

Commit message: Added libraries for electronics
Parts:
- TP1: footprint Connectors:1pin -> Pin_Headers:Pin_Header_Straight_1x01_Pitch2.54mm
Changed lines of the file:
@@
 F 0 "TP1" H 8000 4500 50  0000 C BNN
 F 1 "TEST" H 8000 4450 50  0000 C CNN
-F 2 "Connectors:1pin" H 8000 4200 50  0001 C CNN
+F 2 "Pin_Headers:Pin_Header_Straight_1x01_Pitch2.54mm" H 8000 4200 50  0001 C CNN
 F 3 "" H 8000 4200 50  0001 C CNN
 	1    8000 4200
