Commit message: massive update in observability, now accounts for camera parameters and drone position

File: libraries/tum_simulator/cvg_sim_gazebo/urdf/quadrotor_sensors.urdf.xacro (robot description, xacro)
@@ -22,10 +22,10 @@
     <!-- Forward facing camera -->
     <xacro:include filename="$(find cvg_sim_gazebo)/urdf/sensors/generic_camera.urdf.xacro" />
-    <xacro:generic_camera name="front" sim_name="ardrone" parent="base_link" update_rate="60" res_x="640" res_y="360" image_format="R8G8B8" hfov="${81*M_PI/180}">
+    <xacro:generic_camera name="front" sim_name="ardrone" parent="base_link" update_rate="60" res_x="640" res_y="360" image_format="R8G8B8" hfov="${81*M_PI/180}" tf_prefix="$(arg tf_prefix)">
       <origin xyz="0.21 0.0 0.01" rpy="0 0 0"/>
     </xacro:generic_camera>
     <!-- Downward facing camera -->
     <xacro:include filename="$(find cvg_sim_gazebo)/urdf/sensors/generic_camera.urdf.xacro" />
-    <xacro:generic_camera name="bottom" sim_name="ardrone" parent="base_link" update_rate="60" res_x="640" res_y="360" image_format="R8G8B8" hfov="${81*M_PI/180}">
+    <xacro:generic_camera name="bottom" sim_name="ardrone" parent="base_link" update_rate="60" res_x="640" res_y="360" image_format="R8G8B8" hfov="${81*M_PI/180}" tf_prefix="$(arg tf_prefix)">
         <origin xyz="0.15 0.0 0.0" rpy="0 ${M_PI/2} 0"/>
     </xacro:generic_camera>

File: libraries/tum_simulator/cvg_sim_gazebo/urdf/sensors/generic_camera.urdf.xacro (robot description, xacro)
@@ -4,5 +4,5 @@
 xmlns:xacro="http://ros.org/wiki/xacro">
     <xacro:property name="M_PI" value="3.1415926535897931" />
-    <xacro:macro name="generic_camera" params="name sim_name parent *origin update_rate res_x res_y image_format hfov">
+    <xacro:macro name="generic_camera" params="name sim_name parent *origin update_rate res_x res_y image_format hfov tf_prefix:=''">
       <joint name="${name}_joint" type="fixed">
         <xacro:insert_block name="origin" />
@@ -79,5 +79,5 @@
           <imageTopicName>/${sim_name}/${name}/image_raw</imageTopicName>
           <cameraInfoTopicName>/${sim_name}/${name}/camera_info</cameraInfoTopicName>
-          <frameName>ardrone_base_${name}cam</frameName>
+		  <frameName>${tf_prefix}/ardrone_base_${name}cam</frameName>
         </plugin>
       </sensor>
